Commit message: fix

File: ROS2_Packages/Simulation/simulation_pkg/urdf/arm.urdf.xacro (robot description, xacro)
@@ -1,48 +1,26 @@
 <?xml version="1.0"?>
 <robot xmlns:xacro="http://www.ros.org/wiki/xacro" name="arm">
-<xacro:include filename="$(find sim_pkg_arm)/urdf/arm_joint/arm_joint.urdf.xacro"/>
-<xacro:include filename="$(find sim_pkg_arm)/urdf/arm_part/arm_part.urdf.xacro"/>
-  <!-- Base link -->
-  <link name="base_link">
-    <visual>
-      <geometry>
-        <box size="0.05 0.05 0.02"/>
-      </geometry>
-      <material name="gray">
-        <color rgba="0.5 0.5 0.5 1"/>
-      </material>
-    </visual>
-  </link>
-  <!-- Create the 5 arm links and joints -->
-  <xacro:arm_joint index="1" parent="base_link" child="link1" length="0.05"/>
-  <xacro:arm_part index="1" length="0.05"/>
-  <xacro:arm_joint index="2" parent="link1" child="link2" length="0.04"/>
-  <xacro:arm_part index="2" length="0.05"/>
-  <xacro:arm_joint index="3" parent="link2" child="link3" length="0.035"/>
-  <xacro:arm_part index="3" length="0.05"/>
-  <xacro:arm_joint index="4" parent="link3" child="link4" length="0.03"/>
-  <xacro:arm_part index="4" length="0.05"/>
-  <xacro:arm_joint index="5" parent="link4" child="link5" length="0.025"/>
-  <xacro:arm_part index="5" length="0.025"/>
-  <xacro:gripper_joint parent="5" length="0.05"/>
-  <xacro:gripper_link/>
-  <!-- Add the gripper joint and part -->
-  <!-- <joint name="gripper_joint" type="revolute">
-    <parent link="link5"/>
-    <child link="gripper_link"/>
-    <origin xyz="0 0 0.02" rpy="0 0 0"/>
-    <axis xyz="0 1 0"/>
-    <limit effort="1.0" velocity="1.0" lower="0" upper="0.5"/>
-  </joint>
-  <link name="gripper_link">
-    <visual>
-      <geometry>
-        <box size="0.04 0.01 0.02"/>
-      </geometry>
-      <origin xyz="0 0 0.01" rpy="0 0 0"/>
-      <material name="green">
-        <color rgba="0 1 0 1"/>
-      </material>
-    </visual>
-  </link> -->
+<xacro:include filename="$(find simulation_pkg)/urdf/arm_joint/arm_joint.urdf.xacro"/>
+<xacro:include filename="$(find simulation_pkg)/urdf/arm_part/arm_part.urdf.xacro"/>
+    <link name="base_link">
+      <visual>
+        <geometry><box size="0.05 0.05 0.01"/></geometry>
+        <origin xyz="0 0 0" rpy="0 0 0"/>
+        <material name="gray"><color rgba="0.3 0.3 0.3 1"/></material>
+      </visual>
+    </link>
+    <!-- 每一段 link 与 joint -->
+    <xacro:arm_part index="1" length="0.06"/>
+    <xacro:arm_joint index="1" parent="base_link" child="link1" length="0.01"/>
+    <xacro:arm_part index="2" length="0.06"/>
+    <xacro:arm_joint index="2" parent="link1" child="link2" length="0.06"/>
+    <xacro:arm_part index="3" length="0.05"/>
+    <xacro:arm_joint index="3" parent="link2" child="link3" length="0.05"/>
+    <xacro:arm_part index="4" length="0.05"/>
+    <xacro:arm_joint index="4" parent="link3" child="link4" length="0.05"/>
+    <xacro:arm_part index="5" length="0.04"/>
+    <xacro:arm_joint index="5" parent="link4" child="link5" length="0.04"/>
+    <!-- 爪子 -->
+    <xacro:gripper_link/>
+    <xacro:gripper_joint parent="link5" length="0.04"/>
 </robot>

File: ROS2_Packages/Simulation/simulation_pkg/urdf/arm_joint/arm_joint.urdf.xacro (robot description, xacro)
@@ -2,11 +2,11 @@
 <robot xmlns:xacro="http://www.ros.org/wiki/xacro">
 <!-- 左右 -->
-  <xacro:macro name="arm_joint" params="index parent child length">
+  <xacro:macro name="arm_joint" params="index parent child length rpy='0 0 0' axis='0 0 1' lower='-1.57' upper='1.57'">
     <joint name="joint${index}" type="revolute">
       <parent link="${parent}"/>
       <child link="${child}"/>
-      <origin xyz="0 0 ${length}" rpy="0 0 0"/>
-      <axis xyz="0 0 1"/>
-      <limit lower="-1.57" upper="1.57" effort="1.0" velocity="1.0"/>
+      <origin xyz="0 0 ${length}" rpy="${rpy}"/>
+      <axis xyz="${axis}"/>
+      <limit effort="1.0" velocity="1.0" lower="${lower}" upper="${upper}"/>
     </joint>
   </xacro:macro>
@@ -14,5 +14,5 @@
   <xacro:macro name="gripper_joint" params="parent length">
     <joint name="gripper_joint" type="revolute">
-      <parent link="link${parent}"/>
+      <parent link="${parent}"/>
       <child link="gripper_link"/>
       <origin xyz="0 0 ${length}" rpy="0 0 0"/>

File: ROS2_Packages/Simulation/simulation_pkg/urdf/arm_part/arm_part.urdf.xacro (robot description, xacro)
@@ -1,15 +1,14 @@
 <?xml version="1.0"?>
 <robot xmlns:xacro="http://www.ros.org/wiki/xacro">
-  <xacro:macro name="arm_part" params="index length">
-    <!-- 计算中点 -->
+  <xacro:macro name="arm_part" params="index length radius:=0.01 color:='0 0 1 1'">
     <xacro:property name="half_length" value="${0.5 * length}"/>
     <link name="link${index}">
       <visual>
         <geometry>
-          <cylinder length="${length}" radius="0.01"/>
+          <cylinder length="${length}" radius="${radius}"/>
         </geometry>
         <origin xyz="0 0 ${half_length}" rpy="0 0 0"/>
-        <material name="blue">
-          <color rgba="0 0 1 1"/>
+        <material name="color${index}">
+          <color rgba="${color}"/>
         </material>
       </visual>
